File: sensor_node_v0.03.sch (EAGLE design)
At the start: 50 parts, among them IC1 MCP1703CB, IC2 MCP1703CB, Q1 MMBT5088-NPN, U1 ATMEGA328P_TQFP, U2 TSL2561FN, U4 MPL115A, Y1 16MHZ

Commit message: Replaced mic
Parts:
- removed C11: 100pF, SparkFun-Passives:CAP0805
- removed MIC: (no value), microbuilder:ELECTRET
- removed R10, R11, R9: 1K, SparkFun-Passives:RESISTOR0805-RES
- removed R12: 22K, SparkFun-Passives:RESISTOR0805-RES
- removed TRIMPOT: (no value), microbuilder:TRIMPOTTC33X-2
- removed U3: (no value), microbuilder:MAX4466""
- added C2: 100pF, SparkFun-Capacitors:CAP0805
- added R1: 10K, SparkFun-Passives:RESISTOR0805-RES
- added R3: 1.5K, SparkFun-Passives:RESISTOR0805-RES
- added U$2: ADMP401, SparkFun-Sensors:ADMP401
- added U$3: OPA344, SparkFun-AnalogIC:OPA344
- C10: value 10uF -> 0.1uF; device SparkFun-Passives:CAP0805 -> SparkFun-Capacitors:CAP0805; OC_NEWARK (none) -> unknown
- C8: value 0.01uF -> 4.7uF; device SparkFun-Passives:CAP0805 -> SparkFun-Capacitors:CAP0805; OC_NEWARK (none) -> unknown
- C9: value 0.1uF -> 1uF; device SparkFun-Passives:CAP0805 -> SparkFun-Capacitors:CAP0805; OC_NEWARK (none) -> unknown
- R7: value 1M -> 10K; OC_NEWARK (none) -> unknown
- R8: value 1M -> 100K; OC_NEWARK (none) -> unknown
Connections:
- removed net N$15: C10.1, R11.1
- removed net N$16: R12.2, TRIMPOT.E
- removed net N$6: C8.2, R7.1, R8.2, U3.IN+
- new net N$11: C9.1, R1.2, R7.1, U$3.+IN
- new net SS: J2.9, U1.PB2(SS/OC1B)
- net A0: now also C2.2, R8.1, U$3.OUT; no longer C11.2, TRIMPOT.A, U3.OUT
- net GND0: now also R1.1, U$2.GND@2, U$2.GND@4, U$2.GND@6, U$3.V-; no longer MIC.1, R8.1, U3.GND
- net N$10: now also C2.1, R3.1, R8.2, U$3.-IN; no longer C9.1, R10.1, R9.2
- net N$7: now also C8.1, U$2.OUT; no longer C11.1, R11.2, R12.1, U3.IN-
- net N$9: now also C8.2, R3.2; no longer C8.1, MIC.2, R9.1
- net VCC: now also C10.1, U$2.VDD, U$3.V+; no longer R10.2, U3.VCC
Other:
- note added: "Designed by Akram Ali and Dave Conrod"
- note added: "v0.3 (September 2016)"
- note removed: "Designed by Akram Ali"
- note removed: "v0.1 (July 2016)"
- moved on the sheet: C10, C8, C9, LED2, R4, R7, R8

Commit message: Added RFM69 pads, FTDI chip, USB-microB, bug fixes
Parts:
- added C11: 0.1uF, SparkFun-Capacitors:CAP0805
- added J3: USB-MICROB, SparkFun-Connectors:USB-MICROB
- added LED1, LED3: (no value), adafruit:LEDCHIPLED_0805
- added R10, R9: 47, SparkFun-Passives:RESISTOR0805-RES
- added R11: SHOTTKY, SparkFun-Passives:RESISTOR0805-RES
- added R12, R21: 27, SparkFun-Passives:RESISTOR0805-RES
- added U$4: LOWPOWERLAB_RFM69, RFM69 USB Gateway:LOWPOWERLAB_RFM69
- added U5: FT231XS, SparkFun-DigitalIC:FT231XS
Connections:
- new net ANT: U$4.ANT
- new net D2: U$4.DIO0, U1.PD2(INT0)
- new net FTDI_VCC: R10.1, R9.1, U5.!RESET, U5.3V3OUT, U5.VCCIO
- new net N$17: LED1.C, U5.CBUS1
- new net N$18: LED3.C, U5.CBUS2
- new net N$24: C11.1, J3.VBUS, R11.2, U5.VCC
- new net N$25: R21.1, U5.USBDM
- new net N$26: R12.1, U5.USBDP
- new net N$27: LED1.A, R9.2
- new net N$29: LED3.A, R10.2
- new net N$32: J3.D-, R21.2
- new net N$33: J3.D+, R12.2
- net DTR: now also U5.!DTR
- net GND: now also C11.2, J3.GND, U$4.GND, U5.GND@16, U5.GND@6
- net MISO: now also U$4.MISO
- net MOSI: now also U$4.MOSI
- net PWR: now also R11.1
- net RX: now also U5.TXD
- net SCK: now also U$4.SCK
- net SS: now also U$4.SEL
- net TX: now also U5.RXD
- net VCC: now also U$4.VCC
Other:
- note added: "RFM69HW"
- note added: "USB + FTDI"
- moved on the sheet: C10, C16, C17, C2, C4, C5, C8, C9, IAQ-CORE, IC2, R1, R3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

Commit message: Changed font size of labels
Parts:
- U$4: value LOWPOWERLAB_RFM69 -> RFM69HW
- U1: value ATMEGA328P_TQFP -> ATMEGA328P
Changed lines of the file:
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@@
 </classes>
 <parts>
-<part name="U1" library="SparkFun-DigitalIC" deviceset="ATMEGA328P_TQFP" device="" value="ATMEGA328P_TQFP">
+<part name="U1" library="SparkFun-DigitalIC" deviceset="ATMEGA328P_TQFP" device="" value="ATMEGA328P">
 <attribute name="MF" value=""/>
 <attribute name="MPN" value="ATMEGA328PB-AU"/>
@@
 <part name="GND9" library="SparkFun-Aesthetics" deviceset="GND" device=""/>
 <part name="GND10" library="SparkFun-Aesthetics" deviceset="GND" device=""/>
-<part name="U$4" library="RFM69 USB Gateway" deviceset="LOWPOWERLAB_RFM69" device=""/>
+<part name="U$4" library="RFM69 USB Gateway" deviceset="LOWPOWERLAB_RFM69" device="" value="RFM69HW"/>
 </parts>
 <sheets>
