File: hardware/SensorBoard/v0.4/sensor_board_v0.4.brd (EAGLE design)
At the start: 46.8 x 39.9 mm, 59 parts, among them IC1 MCP1703CB, IC2 MCP1703CB, J3 USB-MICROB, Q1 MMBT5088-NPN, U1 ATMEGA328P, U2 TSL2561FN, U4 MPL115A, U5 FT231XS, Y1 16MHZ

Commit message: Minor touches
Parts:
- moved X1 4.01 mm to (52.3, 42.8), turned to 180 degrees
Routing:
- net PRE: track 35.6 -> 36.3 mm
Other:
- board text removed: "bruh"
