File: hardware/SensorBoard/v0.5/sensor_board_v0.5.sch (EAGLE design)
At the start: 59 parts, among them IC1 MCP1703CB, IC2 MCP1703CB, J3 USB-MICROB, Q1 MMBT5088, U1 ATMEGA328P, U2 TSL2561FN, U4 MPL115A, U5 FT231XS, Y1 16MHZ

Commit message: Removed NPN transistor
connected everything to common GND
Parts:
- removed Q1: MMBT5088, SparkFun-DiscreteSemi:TRANSISTOR_NPNMMBT5088
- removed R2: 330, SparkFun-Passives:RESISTOR0805-RES
Connections:
- removed net GND0: C10.2, C13.2, C14.2, C16.2, C17.2, C3.2, C4.2, C5.2, C7.2, C9.2, IAQ-CORE.GND, IC2.GND, MOSFET.S, Q1.C, R1.1, R14.1, R15.1, R16.1, R17.1, R19.1, U$1.ADDR, U$1.GND, U$1.NC, U$2.GND@2, U$2.GND@4, U$2.GND@6, U$3.V-, U2.GND, U4.GND, X1.GND1, X1.GND2, X1.GND3, X1.GND4
- removed net N$1: Q1.B, R2.2
- net D5: no longer R2.1
- net GND: now also C10.2, C13.2, C14.2, C16.2, C17.2, C3.2, C4.2, C5.2, C7.2, C9.2, IAQ-CORE.GND, IC2.GND, MOSFET.S, R1.1, R14.1, R15.1, R16.1, R17.1, R19.1, U$1.ADDR, U$1.GND, U$1.NC, U$2.GND@2, U$2.GND@4, U$2.GND@6, U$3.V-, U2.GND, U4.GND, X1.GND1, X1.GND2, X1.GND3, X1.GND4; no longer Q1.E
Other:
- note added: "v0.5 (September 2016)"
- note removed: "NPN transistor"
- note removed: "v0.3 (September 2016)"
- moved on the sheet: C16, C17, IC2

Commit message: Increased thickness of power lines to 16
Connections:
- net N$24 renamed VBUS
Changed lines of the file:
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@@
 </segment>
 </net>
-<net name="N$24" class="0">
+<net name="VBUS" class="0">
 <segment>
 <pinref part="U5" gate="U$1" pin="VCC"/>

Commit message: Added I2C addresses in schematic
Parts:
- renumbered IC1 to U8, IC2 to U9, U$1 to U7, U$2 to U6
Other:
- note added: "0x39"
- note added: "0x44"
- note added: "0x5A"
- note added: "0x60"
Changed lines of the file:
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@@
 <attribute name="OC_NEWARK" value="58Y6083"/>
 </part>
-<part name="U$1" library="thomasb9511" deviceset="SHT31-DIS" device="">
+<part name="U7" library="thomasb9511" deviceset="SHT31-DIS" device="">
 <attribute name="MF" value=""/>
 <attribute name="MPN" value="SHT31-DIS-B"/>
@@
 </part>
 <part name="GND8" library="SparkFun-Aesthetics" deviceset="GND" device=""/>
-<part name="IC1" library="linear" deviceset="MCP1703" device="CB">
+<part name="U8" library="linear" deviceset="MCP1703" device="CB">
 <attribute name="MF" value=""/>
 <attribute name="MPN" value="MCP1703T-2502E/CB"/>
@@
 <attribute name="OC_NEWARK" value="unknown"/>
 </part>
-<part name="IC2" library="linear" deviceset="MCP1703" device="CB">
+<part name="U9" library="linear" deviceset="MCP1703" device="CB">
 <attribute name="MF" value=""/>
 <attribute name="MPN" value="MCP1703T-2502E/CB"/>
@@
 <attribute name="OC_NEWARK" value="unknown"/>
 </part>
-<part name="U$2" library="SparkFun-Sensors" deviceset="ADMP401" device=""/>
+<part name="U6" library="SparkFun-Sensors" deviceset="ADMP401" device=""/>
 <part name="U$3" library="SparkFun-AnalogIC" deviceset="OPA344" device=""/>
 <part name="C2" library="SparkFun-Capacitors" deviceset="CAP" device="0805" value="100pF">
@@
 <text x="68.58" y="58.42" size="3.81" layer="94">RFM69HW</text>
 <text x="60.96" y="-17.78" size="3.81" layer="94">USB + FTDI</text>
+<text x="68.58" y="86.36" size="1.778" layer="97">0x39</text>
+<text x="165.1" y="91.44" size="1.778" layer="97">0x60</text>
+<text x="187.96" y="5.08" size="1.778" layer="97">0x5A</text>
+<text x="309.88" y="-30.48" size="1.778" layer="97">0x44</text>
 </plain>
 <instances>
@@
 <attribute name="MPN" x="281.94" y="81.28" size="1.778" layer="96" rot="R270" display="off"/>
 </instance>
-<instance part="U$1" gate="G$1" x="304.8" y="-17.78">
+<instance part="U7" gate="G$1" x="304.8" y="-17.78">
 <attribute name="OC_NEWARK" x="304.8" y="-17.78" size="1.778" layer="96" rot="R270" display="off"/>
 <attribute name="MF" x="304.8" y="-17.78" size="1.778" layer="96" rot="R270" display="off"/>
@@
 </instance>
 <instance part="GND8" gate="1" x="347.98" y="60.96"/>
-<instance part="IC1" gate="G$1" x="-30.48" y="35.56">
+<instance part="U8" gate="G$1" x="-30.48" y="35.56">
 <attribute name="OC_NEWARK" x="-30.48" y="35.56" size="1.778" layer="96" rot="R270" display="off"/>
 <attribute name="MF" x="-30.48" y="35.56" size="1.778" layer="96" rot="R270" display="off"/>
@@
 <attribute name="MPN" x="81.28" y="-119.38" size="1.778" layer="96" rot="R270" display="off"/>
 </instance>
-<instance part="IC2" gate="G$1" x="-30.48" y="-38.1">
+<instance part="U9" gate="G$1" x="-30.48" y="-38.1">
 <attribute name="OC_NEWARK" x="-30.48" y="-38.1" size="1.778" layer="96" rot="R270" display="off"/>
 <attribute name="MF" x="-30.48" y="-38.1" size="1.778" layer="96" rot="R270" display="off"/>
@@
 <attribute name="MPN" x="2.54" y="-48.26" size="1.778" layer="96" rot="R270" display="off"/>
 </instance>
-<instance part="U$2" gate="G$1" x="274.32" y="-119.38"/>
+<instance part="U6" gate="G$1" x="274.32" y="-119.38"/>
 <instance part="U$3" gate="G$1" x="327.66" y="-121.92"/>
 <instance part="C2" gate="G$1" x="330.2" y="-91.44" rot="R90">
@@
 <wire x1="-60.96" y1="22.86" x2="-60.96" y2="20.32" width="0.1524" layer="91"/>
 <wire x1="-60.96" y1="20.32" x2="-30.48" y2="20.32" width="0.1524" layer="91"/>
-<pinref part="IC1" gate="G$1" pin="GND"/>
+<pinref part="U8" gate="G$1" pin="GND"/>
 <wire x1="-30.48" y1="20.32" x2="-30.48" y2="27.94" width="0.1524" layer="91"/>
 <wire x1="-30.48" y1="20.32" x2="2.54" y2="20.32" width="0.1524" layer="91"/>
@@
 <wire x1="-60.96" y1="-50.8" x2="-60.96" y2="-53.34" width="0.1524" layer="91"/>
 <wire x1="-60.96" y1="-53.34" x2="-30.48" y2="-53.34" width="0.1524" layer="91"/>
-<pinref part="IC2" gate="G$1" pin="GND"/>
+<pinref part="U9" gate="G$1" pin="GND"/>
 <wire x1="-30.48" y1="-53.34" x2="-30.48" y2="-45.72" width="0.1524" layer="91"/>
 <wire x1="-30.48" y1="-53.34" x2="2.54" y2="-53.34" width="0.1524" layer="91"/>
@@
 </segment>
 <segment>
-<pinref part="U$2" gate="G$1" pin="GND@2"/>
+<pinref part="U6" gate="G$1" pin="GND@2"/>
 <wire x1="264.16" y1="-121.92" x2="261.62" y2="-121.92" width="0.1524" layer="91"/>
 <wire x1="261.62" y1="-121.92" x2="261.62" y2="-124.46" width="0.1524" layer="91"/>
-<pinref part="U$2" gate="G$1" pin="GND@4"/>
+<pinref part="U6" gate="G$1" pin="GND@4"/>
 <wire x1="261.62" y1="-124.46" x2="264.16" y2="-124.46" width="0.1524" layer="91"/>
-<pinref part="U$2" gate="G$1" pin="GND@6"/>
+<pinref part="U6" gate="G$1" pin="GND@6"/>
 <wire x1="264.16" y1="-127" x2="261.62" y2="-127" width="0.1524" layer="91"/>
 <wire x1="261.62" y1="-127" x2="261.62" y2="-124.46" width="0.1524" layer="91"/>
@@
 </segment>
 <segment>
-<pinref part="U$1" gate="G$1" pin="GND"/>
+<pinref part="U7" gate="G$1" pin="GND"/>
 <wire x1="320.04" y1="-10.16" x2="325.12" y2="-10.16" width="0.1524" layer="91"/>
 <label x="332.74" y="-10.16" size="1.778" layer="95" xref="yes"/>
-<pinref part="U$1" gate="G$1" pin="NC"/>
+<pinref part="U7" gate="G$1" pin="NC"/>
 <wire x1="325.12" y1="-10.16" x2="332.74" y2="-10.16" width="0.1524" layer="91"/>
 <wire x1="320.04" y1="-15.24" x2="325.12" y2="-15.24" width="0.1524" layer="91"/>
@@
 </segment>
 <segment>
-<pinref part="U$1" gate="G$1" pin="ADDR"/>
+<pinref part="U7" gate="G$1" pin="ADDR"/>
 <wire x1="289.56" y1="-15.24" x2="284.48" y2="-15.24" width="0.1524" layer="91"/>
 <label x="284.48" y="-15.24" size="1.778" layer="95" rot="R180" xref="yes"/>
@@
 </segment>
 <segment>
-<pinref part="U$1" gate="G$1" pin="VCC"/>
+<pinref part="U7" gate="G$1" pin="VCC"/>
 <wire x1="320.04" y1="-25.4" x2="327.66" y2="-25.4" width="0.1524" layer="91"/>
 <pinref part="C4" gate="G$1" pin="1"/>
@@
 </segment>
 <segment>
-<pinref part="IC1" gate="G$1" pin="VO"/>
+<pinref part="U8" gate="G$1" pin="VO"/>
 <pinref part="C6" gate="G$1" pin="1"/>
 <wire x1="-20.32" y1="35.56" x2="2.54" y2="35.56" width="0.1524" layer="91"/>
@@
 </segment>
 <segment>
-<pinref part="U$2" gate="G$1" pin="VDD"/>
+<pinref part="U6" gate="G$1" pin="VDD"/>
 <pinref part="C10" gate="G$1" pin="1"/>
 <wire x1="264.16" y1="-111.76" x2="254" y2="-111.76" width="0.1524" layer="91"/>
@@
 </segment>
 <segment>
-<pinref part="U$1" gate="G$1" pin="SCL"/>
+<pinref part="U7" gate="G$1" pin="SCL"/>
 <wire x1="289.56" y1="-25.4" x2="280.67" y2="-25.4" width="0.1524" layer="91"/>
 <label x="280.67" y="-25.4" size="1.778" layer="95" rot="R180" xref="yes"/>
@@
 </segment>
 <segment>
-<pinref part="U$1" gate="G$1" pin="SDA"/>
+<pinref part="U7" gate="G$1" pin="SDA"/>
 <wire x1="289.56" y1="-10.16" x2="280.67" y2="-10.16" width="0.1524" layer="91"/>
 <label x="280.67" y="-10.16" size="1.778" layer="95" rot="R180" xref="yes"/>
@@
 <net name="PWR" class="0">
 <segment>
-<pinref part="IC1" gate="G$1" pin="VI"/>
+<pinref part="U8" gate="G$1" pin="VI"/>
 <pinref part="C1" gate="G$1" pin="1"/>
 <wire x1="-40.64" y1="35.56" x2="-60.96" y2="35.56" width="0.1524" layer="91"/>
@@
 </segment>
 <segment>
-<pinref part="IC2" gate="G$1" pin="VI"/>
+<pinref part="U9" gate="G$1" pin="VI"/>
 <pinref part="C16" gate="G$1" pin="1"/>
 <wire x1="-40.64" y1="-38.1" x2="-60.96" y2="-38.1" width="0.1524" layer="91"/>
@@
 </segment>
 <segment>
-<pinref part="IC2" gate="G$1" pin="VO"/>
+<pinref part="U9" gate="G$1" pin="VO"/>
 <pinref part="C17" gate="G$1" pin="1"/>
 <wire x1="-20.32" y1="-38.1" x2="2.54" y2="-38.1" width="0.1524" layer="91"/>
@@
 <net name="N$7" class="0">
 <segment>
-<pinref part="U$2" gate="G$1" pin="OUT"/>
+<pinref part="U6" gate="G$1" pin="OUT"/>
 <pinref part="C8" gate="G$1" pin="1"/>
 <wire x1="284.48" y1="-119.38" x2="287.02" y2="-119.38" width="0.1524" layer="91"/>

Commit message: Added decoupling cap for ATmega328P
0.1uF
Parts:
- added C15: 0.1uF, SparkFun-Passives:CAP0805
Connections:
- net GND: now also C15.2
- net VCC: now also C15.1
Changed lines of the file:
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@@
 <part name="U$4" library="RFM69 USB Gateway" deviceset="LOWPOWERLAB_RFM69" device="" value="RFM69HW"/>
 <part name="X1" library="adafruit" deviceset="SMACONNECTOR" device="_EDGE"/>
+<part name="C15" library="SparkFun-Passives" deviceset="CAP" device="0805" value="0.1uF"/>
 </parts>
 <sheets>
@@
 <instance part="U$4" gate="G$1" x="81.28" y="27.94"/>
 <instance part="X1" gate="G$1" x="124.46" y="30.48"/>
+<instance part="C15" gate="G$1" x="236.22" y="76.2"/>
 </instances>
 <busses>
@@
 <wire x1="251.46" y1="68.58" x2="251.46" y2="60.96" width="0.1524" layer="91"/>
 <junction x="251.46" y="60.96"/>
+<pinref part="C15" gate="G$1" pin="2"/>
+<wire x1="236.22" y1="73.66" x2="236.22" y2="60.96" width="0.1524" layer="91"/>
+<wire x1="236.22" y1="60.96" x2="251.46" y2="60.96" width="0.1524" layer="91"/>
 </segment>
 <segment>
@@
 <wire x1="251.46" y1="106.68" x2="251.46" y2="127" width="0.1524" layer="91"/>
 <junction x="251.46" y="106.68"/>
+<pinref part="C15" gate="G$1" pin="1"/>
+<wire x1="251.46" y1="101.6" x2="236.22" y2="101.6" width="0.1524" layer="91"/>
+<wire x1="236.22" y1="101.6" x2="236.22" y2="81.28" width="0.1524" layer="91"/>
+<junction x="251.46" y="101.6"/>
 </segment>
 <segment>
@@
 <wire x1="256.54" y1="111.76" x2="243.84" y2="111.76" width="0.1524" layer="91"/>
 <pinref part="R13" gate="G$1" pin="1"/>
-<wire x1="243.84" y1="111.76" x2="236.22" y2="111.76" width="0.1524" layer="91"/>
 <wire x1="243.84" y1="114.3" x2="243.84" y2="111.76" width="0.1524" layer="91"/>
 <junction x="243.84" y="111.76"/>
-<wire x1="236.22" y1="106.68" x2="236.22" y2="111.76" width="0.1524" layer="91"/>
 <pinref part="RESET" gate="S" pin="4"/>
 <wire x1="223.52" y1="111.76" x2="228.6" y2="111.76" width="0.1524" layer="91"/>
-<junction x="236.22" y="111.76"/>
 <pinref part="C12" gate="G$1" pin="2"/>
 <wire x1="228.6" y1="111.76" x2="236.22" y2="111.76" width="0.1524" layer="91"/>
+<wire x1="236.22" y1="111.76" x2="243.84" y2="111.76" width="0.1524" layer="91"/>
 <wire x1="228.6" y1="116.84" x2="228.6" y2="114.3" width="0.1524" layer="91"/>
 <junction x="228.6" y="111.76"/>
@@
 <wire x1="228.6" y1="114.3" x2="223.52" y2="114.3" width="0.1524" layer="91"/>
 <junction x="228.6" y="114.3"/>
-<label x="236.22" y="106.68" size="1.778" layer="95" rot="R270" xref="yes"/>
-</segment>
-<segment>
+<label x="228.6" y="101.6" size="1.778" layer="95" rot="R270" xref="yes"/>
+<wire x1="228.6" y1="101.6" x2="228.6" y2="104.14" width="0.1524" layer="91"/>
+<wire x1="228.6" y1="104.14" x2="236.22" y2="111.76" width="0.1524" layer="91"/>
+<junction x="236.22" y="111.76"/>
+</segment>
+<segment>

Commit message: Moved decoupling caps closer to ICs
Parts:
- U2: value TSL2561FN -> TSL2561
Changed lines of the file:
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@@
 <attribute name="OC_NEWARK" value="47Y1304"/>
 </part>
-<part name="U2" library="SparkFun-DigitalIC" deviceset="TSL2561" device="FN">
+<part name="U2" library="SparkFun-DigitalIC" deviceset="TSL2561" device="FN" value="TSL2561">
 <attribute name="DIGIKEY#" value="TSL2561-FNCT-ND"/>
 <attribute name="MANF" value="AMS-TAOS-USA-Inc."/>

Commit message: Moved Trace on PiAQ, v4 of enclosure
Parts:
- C13: OC_NEWARK (none) -> unknown
Changed lines of the file:
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@@
 <part name="J2" library="SparkFun-Connectors" deviceset="M05X2" device="PTH"/>
 <part name="U4" library="SparkFun-Sensors" deviceset="MPL115A" device=""/>
-<part name="C13" library="SparkFun-Passives" deviceset="CAP" device="0805" value="0.1uF"/>
+<part name="C13" library="SparkFun-Passives" deviceset="CAP" device="0805" value="0.1uF">
+<attribute name="MF" value=""/>
+<attribute name="MPN" value=""/>
+<attribute name="OC_NEWARK" value="unknown"/>
+</part>
 <part name="C14" library="SparkFun-Passives" deviceset="CAP" device="0805" value="0.1uF"/>
 <part name="SUPPLY12" library="SparkFun-Aesthetics" deviceset="VCC" device=""/>
@@
 <instance part="J2" gate="G$1" x="-33.02" y="111.76"/>
 <instance part="U4" gate="G$1" x="160.02" y="101.6"/>
-<instance part="C13" gate="G$1" x="132.08" y="96.52"/>
+<instance part="C13" gate="G$1" x="132.08" y="96.52">
+<attribute name="MF" x="132.08" y="96.52" size="1.778" layer="96" display="off"/>
+<attribute name="MPN" x="132.08" y="96.52" size="1.778" layer="96" display="off"/>
+<attribute name="OC_NEWARK" x="132.08" y="96.52" size="1.778" layer="96" display="off"/>
+</instance>
 <instance part="C14" gate="G$1" x="124.46" y="96.52"/>
 <instance part="SUPPLY12" gate="G$1" x="124.46" y="111.76"/>
