File: hardware/PiHAT/PiHAT.sch (EAGLE design)
At the start: 41 parts, among them U1 ATMEGA328P, U2 TSL2561, U3 OPA344, U4 MPL115A, U6 ADMP401, U7 SHT31-DIS, Y1 16MHZ

Commit message: continuing to add BOM materials
Parts:
- C10, C3, C4, C5: OC_NEWARK unknown -> (none)
- IAQ-CORE: DIGIKEY# (none) -> IAQ-CORE C-ND
- RESET: DIGIKEY# (none) -> CKN9104CT-ND
- U1: DIGIKEY# (none) -> ATMEGA328P-AU-ND
- U3: DIGIKEY# (none) -> 296-41475-1-ND
- U6: DIGIKEY# (none) -> INMP401ACEZ-R7CT-ND
- U7: DIGIKEY# (none) -> 1649-1011-1-ND
Changed lines of the file:
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@@
 <part name="GND2" library="supply1" deviceset="GND" device=""/>
 <part name="U1" library="SparkFun-DigitalIC" deviceset="ATMEGA328P_TQFP" device="" value="ATMEGA328P">
+<attribute name="DIGIKEY#" value="ATMEGA328P-AU-ND"/>
 <attribute name="MF" value=""/>
 <attribute name="MPN" value="ATMEGA328PB-AU"/>
@@
 </part>
 <part name="U7" library="thomasb9511" deviceset="SHT31-DIS" device="">
+<attribute name="DIGIKEY#" value="1649-1011-1-ND"/>
 <attribute name="MF" value=""/>
 <attribute name="MPN" value="SHT31-DIS-B"/>
@@
 </part>
 <part name="IAQ-CORE" library="IAQ-CORE" deviceset="IAQ-CORE" device="">
+<attribute name="DIGIKEY#" value="IAQ-CORE C-ND"/>
 <attribute name="MF" value=""/>
 <attribute name="MPN" value="IAQ CORE"/>
@@
 <attribute name="OC_NEWARK" value="unknown"/>
 </part>
-<part name="C3" library="SparkFun-Passives" deviceset="CAP" device="0805" value="0.1uF">
-<attribute name="MF" value=""/>
-<attribute name="MPN" value=""/>
-<attribute name="OC_NEWARK" value="unknown"/>
-</part>
-<part name="C4" library="SparkFun-Passives" deviceset="CAP" device="0805" value="0.1uF">
-<attribute name="MF" value=""/>
-<attribute name="MPN" value=""/>
-<attribute name="OC_NEWARK" value="unknown"/>
-</part>
-<part name="C5" library="SparkFun-Passives" deviceset="CAP" device="0805" value="0.1uF">
-<attribute name="MF" value=""/>
-<attribute name="MPN" value=""/>
-<attribute name="OC_NEWARK" value="unknown"/>
-</part>
+<part name="C3" library="SparkFun-Passives" deviceset="CAP" device="0805" value="0.1uF"/>
+<part name="C4" library="SparkFun-Passives" deviceset="CAP" device="0805" value="0.1uF"/>
+<part name="C5" library="SparkFun-Passives" deviceset="CAP" device="0805" value="0.1uF"/>
 <part name="Y1" library="SparkFun-FreqCtrl" deviceset="RESONATOR" device="16MHZ" value="16MHZ">
 <attribute name="MF" value=""/>
@@
 <part name="C12" library="SparkFun-Passives" deviceset="CAP" device="0805" value="0.1uF"/>
 <part name="GND5" library="SparkFun-Aesthetics" deviceset="GND" device=""/>
-<part name="RESET" library="SparkFun-Retired" deviceset="TAC_SWITCH" device="SMD" value="TAC_SWITCHSMD"/>
+<part name="RESET" library="SparkFun-Retired" deviceset="TAC_SWITCH" device="SMD" value="TAC_SWITCHSMD">
+<attribute name="DIGIKEY#" value="CKN9104CT-ND"/>
+</part>
 <part name="SUPPLY11" library="SparkFun-Aesthetics" deviceset="VCC" device=""/>
 <part name="J2" library="SparkFun-Connectors" deviceset="M05X2" device="PTH"/>
@@
 <attribute name="OC_NEWARK" value="unknown"/>
 </part>
-<part name="U6" library="SparkFun-Sensors" deviceset="ADMP401" device=""/>
-<part name="U3" library="SparkFun-AnalogIC" deviceset="OPA344" device=""/>
+<part name="U6" library="SparkFun-Sensors" deviceset="ADMP401" device="">
+<attribute name="DIGIKEY#" value="INMP401ACEZ-R7CT-ND"/>
+</part>
+<part name="U3" library="SparkFun-AnalogIC" deviceset="OPA344" device="">
+<attribute name="DIGIKEY#" value="296-41475-1-ND"/>
+</part>
 <part name="C2" library="SparkFun-Capacitors" deviceset="CAP" device="0805" value="100pF">
 <attribute name="MF" value=""/>
@@
 <attribute name="OC_NEWARK" value="unknown"/>
 </part>
-<part name="C10" library="SparkFun-Capacitors" deviceset="CAP" device="0805" value="0.1uF">
-<attribute name="MF" value=""/>
-<attribute name="MPN" value=""/>
-<attribute name="OC_NEWARK" value="unknown"/>
-</part>
+<part name="C10" library="SparkFun-Capacitors" deviceset="CAP" device="0805" value="0.1uF"/>
 <part name="R1" library="SparkFun-Passives" deviceset="RESISTOR" device="0805-RES" value="10K">
 <attribute name="MF" value=""/>
@@
 <attribute name="MF" x="464.82" y="86.36" size="1.778" layer="96" rot="R270" display="off"/>
 <attribute name="MPN" x="464.82" y="86.36" size="1.778" layer="96" rot="R270" display="off"/>
+<attribute name="DIGIKEY#" x="464.82" y="86.36" size="1.778" layer="96" display="off"/>
 </instance>
 <instance part="U7" gate="G$1" x="462.28" y="-5.08">
@@
 <attribute name="MF" x="462.28" y="-5.08" size="1.778" layer="96" rot="R270" display="off"/>
 <attribute name="MPN" x="462.28" y="-5.08" size="1.778" layer="96" rot="R270" display="off"/>
+<attribute name="DIGIKEY#" x="462.28" y="-5.08" size="1.778" layer="96" display="off"/>
 </instance>
 <instance part="U2" gate="G$1" x="317.5" y="30.48">
@@
 <attribute name="MF" x="345.44" y="-52.07" size="1.778" layer="96" rot="R270" display="off"/>
 <attribute name="MPN" x="345.44" y="-52.07" size="1.778" layer="96" rot="R270" display="off"/>
+<attribute name="DIGIKEY#" x="345.44" y="-52.07" size="1.778" layer="96" display="off"/>
 </instance>
 <instance part="GND3" gate="1" x="434.34" y="53.34"/>
@@
 <attribute name="MPN" x="510.54" y="114.3" size="1.778" layer="96" rot="R270" display="off"/>
 </instance>
-<instance part="C3" gate="G$1" x="337.82" y="30.48">
-<attribute name="OC_NEWARK" x="337.82" y="30.48" size="1.778" layer="96" rot="R270" display="off"/>
-<attribute name="MF" x="337.82" y="30.48" size="1.778" layer="96" rot="R270" display="off"/>
-<attribute name="MPN" x="337.82" y="30.48" size="1.778" layer="96" rot="R270" display="off"/>
-</instance>
-<instance part="C4" gate="G$1" x="485.14" y="-17.78">
-<attribute name="OC_NEWARK" x="485.14" y="-17.78" size="1.778" layer="96" rot="R270" display="off"/>
-<attribute name="MF" x="485.14" y="-17.78" size="1.778" layer="96" rot="R270" display="off"/>
-<attribute name="MPN" x="485.14" y="-17.78" size="1.778" layer="96" rot="R270" display="off"/>
-</instance>
-<instance part="C5" gate="G$1" x="375.92" y="-53.34">
-<attribute name="OC_NEWARK" x="375.92" y="-53.34" size="1.778" layer="96" rot="R270" display="off"/>
-<attribute name="MF" x="375.92" y="-53.34" size="1.778" layer="96" rot="R270" display="off"/>
-<attribute name="MPN" x="375.92" y="-53.34" size="1.778" layer="96" rot="R270" display="off"/>
-</instance>
+<instance part="C3" gate="G$1" x="337.82" y="30.48"/>
+<instance part="C4" gate="G$1" x="485.14" y="-17.78"/>
+<instance part="C5" gate="G$1" x="375.92" y="-53.34"/>
 <instance part="Y1" gate="G$1" x="434.34" y="81.28">
 <attribute name="OC_NEWARK" x="434.34" y="81.28" size="1.778" layer="96" rot="R270" display="off"/>
@@
 <instance part="C12" gate="G$1" x="411.48" y="124.46"/>
 <instance part="GND5" gate="1" x="393.7" y="111.76"/>
-<instance part="RESET" gate="S" x="401.32" y="119.38"/>
+<instance part="RESET" gate="S" x="401.32" y="119.38">
+<attribute name="DIGIKEY#" x="401.32" y="119.38" size="1.778" layer="96" display="off"/>
+</instance>
 <instance part="SUPPLY11" gate="G$1" x="426.72" y="132.08"/>
 <instance part="J2" gate="G$1" x="187.96" y="-10.16"/>
@@
 <attribute name="MPN" x="284.48" y="-99.06" size="1.778" layer="96" rot="R270" display="off"/>
 </instance>
-<instance part="U6" gate="G$1" x="454.66" y="-99.06"/>
-<instance part="U3" gate="G$1" x="508" y="-101.6"/>
+<instance part="U6" gate="G$1" x="454.66" y="-99.06">
+<attribute name="DIGIKEY#" x="454.66" y="-99.06" size="1.778" layer="96" display="off"/>
+</instance>
+<instance part="U3" gate="G$1" x="508" y="-101.6">
+<attribute name="DIGIKEY#" x="508" y="-101.6" size="1.778" layer="96" display="off"/>
+</instance>
 <instance part="C2" gate="G$1" x="510.54" y="-71.12" rot="R90">
 <attribute name="OC_NEWARK" x="510.54" y="-71.12" size="1.778" layer="96" display="off"/>
@@
 <attribute name="MPN" x="485.14" y="-119.38" size="1.778" layer="96" rot="R270" display="off"/>
 </instance>
-<instance part="C10" gate="G$1" x="434.34" y="-99.06">
-<attribute name="OC_NEWARK" x="434.34" y="-99.06" size="1.778" layer="96" rot="R270" display="off"/>
-<attribute name="MF" x="434.34" y="-99.06" size="1.778" layer="96" rot="R270" display="off"/>
-<attribute name="MPN" x="434.34" y="-99.06" size="1.778" layer="96" rot="R270" display="off"/>
-</instance>
+<instance part="C10" gate="G$1" x="434.34" y="-99.06"/>
 <instance part="R1" gate="G$1" x="495.3" y="-116.84" rot="R90">
 <attribute name="OC_NEWARK" x="495.3" y="-116.84" size="1.778" layer="96" display="off"/>

Commit message: Updating BOM
Parts:
- C10, C12, C13, C14, C15, C3, C4, C5: DIGIKEY# (none) -> 311-1088-1-ND
- C2: DIGIKEY# (none) -> 311-1111-1-ND; OC_NEWARK unknown -> (none)
- C7: DIGIKEY# (none) -> 311-1088-1-ND; OC_NEWARK unknown -> (none)
- C8: DIGIKEY# (none) -> 311-1871-1-ND; OC_NEWARK unknown -> (none)
- C9: DIGIKEY# (none) -> 311-1365-1-ND; OC_NEWARK unknown -> (none)
- LED2: DIGIKEY# (none) -> 475-1196-1-ND
- R1, R5, R6, R7: DIGIKEY# (none) -> 311-10KARCT-ND; OC_NEWARK unknown -> (none)
- R13: DIGIKEY# (none) -> 311-10KARCT-ND
- R14: DIGIKEY# (none) -> RHM47KKCT-ND
- R15, R18, R8: DIGIKEY# (none) -> 541-82.0CCT-NDE; OC_NEWARK unknown -> (none)
- R16: DIGIKEY# (none) -> 311-22KARCT-NDE
- R17: DIGIKEY# (none) -> RHM51KCT-ND; OC_NEWARK unknown -> (none)
- R19: DIGIKEY# (none) -> 311-100KCRCT-NDE; OC_NEWARK unknown -> (none)
- R20: DIGIKEY# (none) -> 311-100CRCT-NDE; OC_NEWARK unknown -> (none)
- R3: DIGIKEY# (none) -> YAG1814CT-ND; OC_NEWARK unknown -> (none)
- R4: DIGIKEY# (none) -> 311-47ARCT-ND
- Y1: DIGIKEY# (none) -> 490-1198-1-ND

Commit message: updating descriptions on bom
Parts:
- R15, R18, R8: DIGIKEY# 541-82.0CCT-NDE -> 541-82.0CCT-ND
- R16: DIGIKEY# 311-22KARCT-NDE -> 311-22KARCT-ND
- R19: DIGIKEY# 311-100KCRCT-NDE -> 311-100KCRCT-ND
- R20: DIGIKEY# 311-100CRCT-NDE -> 311-100CRCT-ND
Changed lines of the file:
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@@
 </part>
 <part name="R15" library="SparkFun-Passives" deviceset="RESISTOR" device="0805-RES" value="82">
-<attribute name="DIGIKEY#" value="541-82.0CCT-NDE"/>
+<attribute name="DIGIKEY#" value="541-82.0CCT-ND"/>
 </part>
 <part name="R16" library="SparkFun-Passives" deviceset="RESISTOR" device="0805-RES" value="22K">
-<attribute name="DIGIKEY#" value="311-22KARCT-NDE"/>
+<attribute name="DIGIKEY#" value="311-22KARCT-ND"/>
 <attribute name="MF" value=""/>
 <attribute name="MPN" value=""/>
@@
 </part>
 <part name="R18" library="SparkFun-Passives" deviceset="RESISTOR" device="0805-RES" value="82">
-<attribute name="DIGIKEY#" value="541-82.0CCT-NDE"/>
+<attribute name="DIGIKEY#" value="541-82.0CCT-ND"/>
 </part>
 <part name="R19" library="SparkFun-Passives" deviceset="RESISTOR" device="0805-RES" value="100K">
-<attribute name="DIGIKEY#" value="311-100KCRCT-NDE"/>
+<attribute name="DIGIKEY#" value="311-100KCRCT-ND"/>
 </part>
 <part name="R20" library="SparkFun-Passives" deviceset="RESISTOR" device="0805-RES" value="100">
-<attribute name="DIGIKEY#" value="311-100CRCT-NDE"/>
+<attribute name="DIGIKEY#" value="311-100CRCT-ND"/>
 </part>
 <part name="MOSFET" library="MICS-4514_CO_and_NOx_Sensor_Breakout" deviceset="SPARKFUN-DISCRETESEMI_MOSFET-NCHANNEL" device="BSS138"/>
@@
 </part>
 <part name="R8" library="SparkFun-Passives" deviceset="RESISTOR" device="0805-RES" value="100K">
-<attribute name="DIGIKEY#" value="541-82.0CCT-NDE"/>
+<attribute name="DIGIKEY#" value="541-82.0CCT-ND"/>
 </part>
 <part name="SUPPLY4" library="SparkFun-Aesthetics" deviceset="VCC" device=""/>

Commit message: Added 5x2 header attribute
Digikey part number
Parts:
- J2: DIGIKEY# (none) -> S6105-ND
Changed lines of the file:
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@@
 </part>
 <part name="SUPPLY11" library="SparkFun-Aesthetics" deviceset="VCC" device=""/>
-<part name="J2" library="SparkFun-Connectors" deviceset="M05X2" device="PTH"/>
+<part name="J2" library="SparkFun-Connectors" deviceset="M05X2" device="PTH">
+<attribute name="DIGIKEY#" value="S6105-ND"/>
+</part>
 <part name="U4" library="SparkFun-Sensors" deviceset="MPL115A" device="">
 <attribute name="DIGIKEY#" value="MPL115A2-ND"/>
@@
 </instance>
 <instance part="SUPPLY11" gate="G$1" x="426.72" y="132.08"/>
-<instance part="J2" gate="G$1" x="187.96" y="-10.16"/>
+<instance part="J2" gate="G$1" x="187.96" y="-10.16">
+<attribute name="DIGIKEY#" x="187.96" y="-10.16" size="1.778" layer="96" display="off"/>
+</instance>
 <instance part="U4" gate="G$1" x="325.12" y="109.22">
 <attribute name="DIGIKEY#" x="325.12" y="109.22" size="1.778" layer="96" display="off"/>

Commit message: Updated BOM
Digikey part number for MOSFET
Parts:
- MOSFET: DIGIKEY# (none) -> BSS138-FDICT-ND
Changed lines of the file:
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@@
 <attribute name="DIGIKEY#" value="311-100CRCT-ND"/>
 </part>
-<part name="MOSFET" library="MICS-4514_CO_and_NOx_Sensor_Breakout" deviceset="SPARKFUN-DISCRETESEMI_MOSFET-NCHANNEL" device="BSS138"/>
+<part name="MOSFET" library="MICS-4514_CO_and_NOx_Sensor_Breakout" deviceset="SPARKFUN-DISCRETESEMI_MOSFET-NCHANNEL" device="BSS138">
+<attribute name="DIGIKEY#" value="BSS138-FDICT-ND"/>
+</part>
 <part name="C7" library="SparkFun-Passives" deviceset="CAP" device="0805" value="0.1uF">
 <attribute name="DIGIKEY#" value="311-1088-1-ND"/>
@@
 <attribute name="DIGIKEY#" x="152.4" y="-119.38" size="1.778" layer="96" rot="R180" display="off"/>
 </instance>
-<instance part="MOSFET" gate="G$1" x="175.26" y="-119.38"/>
+<instance part="MOSFET" gate="G$1" x="175.26" y="-119.38">
+<attribute name="DIGIKEY#" x="175.26" y="-119.38" size="1.778" layer="96" display="off"/>
+</instance>
 <instance part="C7" gate="G$1" x="284.48" y="-99.06">
 <attribute name="DIGIKEY#" x="284.48" y="-99.06" size="1.778" layer="96" display="off"/>
