File: hardware/PiHAT/v0.2/PiHAT.sch (EAGLE design)
At the start: 47 parts, among them J1 FTDI, J3 ISP, U1 ATMEGA328P, U2 TSL2561, U3 OPA344, U4 MPL115A, U6 ADMP401, U7 SHT31-DIS, Y1 16MHZ

Commit message: updating sch for cleaner bom
Parts:
- J1: DIGIKEY# (none) -> 768-1129-1-ND
- J3, RPI1: NO_BOM (none) -> TRUE
- LED2: MPN (none) -> LY L29K-H1K2-26-Z; OC_NEWARK unknown -> (none)
- MICS4514: MANF (none) -> SensorTech; MPN (none) -> MiCS-4514
- U8: MANF (none) -> AMS; MPN (none) -> CCS811
- renumbered U$1 to U8
Changed lines of the file:
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@@
 </classes>
 <parts>
-<part name="RPI1" library="microbuilder" deviceset="RASPBERRYPI_BPLUS" device="_HATSLOTS"/>
+<part name="RPI1" library="microbuilder" deviceset="RASPBERRYPI_BPLUS" device="_HATSLOTS">
+<attribute name="NO_BOM" value="TRUE"/>
+</part>
 <part name="GND1" library="supply1" deviceset="GND" device=""/>
 <part name="GND2" library="supply1" deviceset="GND" device=""/>
@@
 <attribute name="DIGIKEY#" value="475-1196-1-ND"/>
 <attribute name="MF" value=""/>
-<attribute name="MPN" value=""/>
-<attribute name="OC_NEWARK" value="unknown"/>
+<attribute name="MPN" value="LY L29K-H1K2-26-Z"/>
 </part>
 <part name="GND8" library="SparkFun-Aesthetics" deviceset="GND" device=""/>
@@
 </part>
 <part name="SUPPLY12" library="SparkFun-Aesthetics" deviceset="VCC" device=""/>
-<part name="MICS4514" library="MICS-4514_CO_and_NOx_Sensor_Breakout" deviceset="SPARKFUN-SENSORS_MICS-4514" device=""/>
+<part name="MICS4514" library="MICS-4514_CO_and_NOx_Sensor_Breakout" deviceset="SPARKFUN-SENSORS_MICS-4514" device="">
+<attribute name="MANF" value="SensorTech"/>
+<attribute name="MPN" value="MiCS-4514"/>
+</part>
 <part name="R14" library="SparkFun-Passives" deviceset="RESISTOR" device="0805-RES" value="47K">
 <attribute name="DIGIKEY#" value="RHM47KKCT-ND"/>
@@
 </part>
 <part name="GND4" library="SparkFun-Aesthetics" deviceset="GND" device=""/>
-<part name="U$1" library="CCS811" deviceset="CCS811" device="-I2C" value="CCS811"/>
+<part name="U8" library="CCS811" deviceset="CCS811" device="-I2C" value="CCS811">
+<attribute name="MANF" value="AMS"/>
+<attribute name="MPN" value="CCS811"/>
+</part>
 <part name="SUPPLY8" library="SparkFun-Aesthetics" deviceset="VCC" device=""/>
 <part name="R9" library="SparkFun-Passives" deviceset="RESISTOR" device="0805-RES" value="100K">
@@
 </part>
 <part name="J1" library="SparkFun-Connectors" deviceset="FTDI_BASIC" device="PTH" value="FTDI">
+<attribute name="DIGIKEY#" value="768-1129-1-ND"/>
 <attribute name="MPN" value="FT231XS-R"/>
 </part>
-<part name="J3" library="SparkFun-Connectors" deviceset="AVR_SPI_PRG_6" device="PTH" value="ISP"/>
+<part name="J3" library="SparkFun-Connectors" deviceset="AVR_SPI_PRG_6" device="PTH" value="ISP">
+<attribute name="NO_BOM" value="TRUE"/>
+</part>
 </parts>
 <sheets>
@@
 </plain>
 <instances>
-<instance part="RPI1" gate="G$1" x="210.82" y="109.22"/>
+<instance part="RPI1" gate="G$1" x="210.82" y="109.22">
+<attribute name="NO_BOM" x="210.82" y="109.22" size="1.778" layer="96" display="off"/>
+</instance>
 <instance part="GND1" gate="1" x="187.96" y="78.74"/>
 <instance part="GND2" gate="1" x="238.76" y="76.2"/>
@@
 <instance part="SUPPLY7" gate="G$1" x="505.46" y="127"/>
 <instance part="LED2" gate="G$1" x="523.24" y="76.2" rot="R90">
-<attribute name="OC_NEWARK" x="523.24" y="76.2" size="1.778" layer="96" rot="R270" display="off"/>
 <attribute name="MF" x="523.24" y="76.2" size="1.778" layer="96" rot="R270" display="off"/>
 <attribute name="MPN" x="523.24" y="76.2" size="1.778" layer="96" rot="R270" display="off"/>
@@
 </instance>
 <instance part="SUPPLY12" gate="G$1" x="289.56" y="119.38"/>
-<instance part="MICS4514" gate="G$1" x="248.92" y="-106.68"/>
+<instance part="MICS4514" gate="G$1" x="248.92" y="-106.68">
+<attribute name="MPN" x="248.92" y="-106.68" size="1.778" layer="96" display="off"/>
+<attribute name="MANF" x="248.92" y="-106.68" size="1.778" layer="96" display="off"/>
+</instance>
 <instance part="R14" gate="G$1" x="218.44" y="-119.38" rot="R90">
 <attribute name="OC_NEWARK" x="218.44" y="-119.38" size="1.778" layer="96" display="off"/>
@@
 </instance>
 <instance part="GND4" gate="1" x="147.32" y="76.2"/>
-<instance part="U$1" gate="G$1" x="337.82" y="-60.96"/>
+<instance part="U8" gate="G$1" x="337.82" y="-60.96">
+<attribute name="MANF" x="337.82" y="-60.96" size="1.778" layer="96" display="off"/>
+<attribute name="MPN" x="337.82" y="-60.96" size="1.778" layer="96" display="off"/>
+</instance>
 <instance part="SUPPLY8" gate="G$1" x="322.58" y="-33.02"/>
 <instance part="R9" gate="G$1" x="322.58" y="-40.64" rot="R270">
@@
 <instance part="J1" gate="G$1" x="187.96" y="-53.34">
 <attribute name="MPN" x="187.96" y="-53.34" size="1.778" layer="96" display="off"/>
-</instance>
-<instance part="J3" gate="G$1" x="180.34" y="20.32"/>
+<attribute name="DIGIKEY#" x="187.96" y="-53.34" size="1.778" layer="96" display="off"/>
+</instance>
+<instance part="J3" gate="G$1" x="180.34" y="20.32">
+<attribute name="NO_BOM" x="180.34" y="20.32" size="1.778" layer="96" display="off"/>
+</instance>
 </instances>
 <busses>
@@
 </segment>
 <segment>
-<pinref part="U$1" gate="G$1" pin="SDA"/>
+<pinref part="U8" gate="G$1" pin="SDA"/>
 <wire x1="368.3" y1="-48.26" x2="378.46" y2="-48.26" width="0.1524" layer="91"/>
 <label x="378.46" y="-48.26" size="1.778" layer="95" xref="yes"/>
@@
 </segment>
 <segment>
-<pinref part="U$1" gate="G$1" pin="SCL"/>
+<pinref part="U8" gate="G$1" pin="SCL"/>
 <wire x1="368.3" y1="-45.72" x2="370.84" y2="-45.72" width="0.1524" layer="91"/>
 <wire x1="370.84" y1="-45.72" x2="373.38" y2="-43.18" width="0.1524" layer="91"/>
@@
 </segment>
 <segment>
-<pinref part="U$1" gate="G$1" pin="GND"/>
+<pinref part="U8" gate="G$1" pin="GND"/>
 <wire x1="350.52" y1="-66.04" x2="350.52" y2="-68.58" width="0.1524" layer="91"/>
 <pinref part="C5" gate="G$1" pin="2"/>
@@
 </segment>
 <segment>
-<pinref part="U$1" gate="G$1" pin="VDD"/>
+<pinref part="U8" gate="G$1" pin="VDD"/>
 <pinref part="SUPPLY5" gate="G$1" pin="VCC"/>
 <wire x1="368.3" y1="-55.88" x2="375.92" y2="-55.88" width="0.1524" layer="91"/>
@@
 <net name="N$16" class="0">
 <segment>
-<pinref part="U$1" gate="G$1" pin="ADDR"/>
+<pinref part="U8" gate="G$1" pin="ADDR"/>
 <pinref part="R9" gate="G$1" pin="2"/>
 <wire x1="332.74" y1="-45.72" x2="322.58" y2="-45.72" width="0.1524" layer="91"/>

Commit message: adding details to aid in fabrication
Parts:
- removed LED_05: (no value), adafruit:LEDCHIPLED_0805
- added LED1: (no value), adafruit:LEDCHIPLED_0805
- C10, C12, C13, C14, C15, C4, C5, C7: MOUSER# (none) -> 603-CC603KRX7R7BB104
- C2: MOUSER# (none) -> 603-CC805JRNPO9BN101
- C3, R20: MOUSER# (none) -> 603-RC0805FR-07100RL
- C8: MOUSER# (none) -> 603-CC805KKX5R8BB475
- C9: MOUSER# (none) -> 603-CC805KKX7R7BB105
- J1: MOUSER# (none) -> 895-FT231XS-R
- LED2: DESCRIPTION (none) -> LED; MOUSER# (none) -> 720-LYL29KH1K226Z
- LED3: DESCRIPTION (none) -> LED; MOUSER# (none) -> 720-LYL29KH1K226Z; OC_NEWARK unknown -> (none)
- MOSFET: MOUSER# (none) -> 621-BSS138-7-F
- R1, R13, R5, R6, R7: MOUSER# (none) -> 603-RC0805JR-0710KL
- R10, R2, R4: MOUSER# (none) -> 603-RC0805JR-0747RL; OC_NEWARK unknown -> (none)
- R14: MOUSER# (none) -> 755-ESR10EZPJ473; OC_NEWARK unknown -> (none)
- R15, R18: MOUSER# (none) -> CRCW080582R0FKEA
- R16: MOUSER# (none) -> 603-RC0805JR-0722KL; OC_NEWARK unknown -> (none)
- R17: MOUSER# (none) -> 755-ESR10EZPJ510
- R19, R8, R9: MOUSER# (none) -> 603-RC0805FR-07100KL
- R3: MOUSER# (none) -> 603-RT0805BRD071K5L
- RESET: MOUSER# (none) -> 611-PTS525SM15SMTR2
- U1: MOUSER# (none) -> 556-ATMEGA328P-AU; OC_NEWARK 58Y6083 -> (none)
- U2: MANF# TSL2561FN -> (none); OC_NEWARK 82Y5564 -> (none)
- U3: MOUSER# (none) -> 595-OPA344NA/3K
- U4: MOUSER# (none) -> 841-MPL115A2
- U7: MOUSER# (none) -> 403-SHT31-DIS-B; OC_NEWARK 47Y1304 -> (none)
- Y1: MOUSER# (none) -> 81-CSTCE16M0V53-R0
- renumbered LED_26 to LED3
Connections:
- net GND: now also LED1.C; no longer LED_05.C
- net N$3: now also LED1.A; no longer LED2.A
- net N$6: now also LED2.A; no longer LED_05.A
Other:
- moved on the sheet: LED2
