File: hardware/SensorBoard/v0.8/sensor_board_v0.8.sch (EAGLE design)
At the start: 48 parts, among them IC1 BMP280, J3 USB-MICROB, U10 CCS811, U11 RFM69HW, U2 TSL2561, U3 ATMEGA328P-MU, U5 FT231XS, U7 SHT31, U8 MCP1703/3.3V, U9 MCP1703CB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

Commit message: Replaced FT231X SSOP with QFN package
New part number: FT231XQ-R
Adjusted several traces for the new package
Parts:
- removed U5: FT231XS, SparkFun-DigitalIC:FT231XS
- added U$1: FT231XQ-R, ftdi_ft231xq-r:FT231XQ-R
Connections:
- net DTR: now also U$1.DTR#; no longer U5.!DTR
- net FTDI_VCC: now also U$1.3V3OUT, U$1.RESET#, U$1.VCCIO; no longer U5.!RESET, U5.3V3OUT, U5.VCCIO
- net GND: now also U$1.GND_13, U$1.GND_21, U$1.GND_3; no longer U5.GND@16, U5.GND@6
- net N$17: now also U$1.CBUS1; no longer U5.CBUS1
- net N$18: now also U$1.CBUS2; no longer U5.CBUS2
- net N$25: now also U$1.USBDM; no longer U5.USBDM
- net N$26: now also U$1.USBDP; no longer U5.USBDP
- net RX: now also U$1.TXD; no longer U5.TXD
- net TX: now also U$1.RXD; no longer U5.RXD
- net VBUS: now also U$1.VCC; no longer U5.VCC
Other:
- note added: "v0.8 (October 2016)"
- note removed: "v0.6 (October 2016)"
Changed lines of the file:
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@@
 <part name="GND3" library="SparkFun-Aesthetics" deviceset="GND" device=""/>
 <part name="J3" library="SparkFun-Connectors" deviceset="USB" device="-MICROB"/>
-<part name="U5" library="SparkFun-DigitalIC" deviceset="FT231X" device="S" value="FT231XS"/>
 <part name="RX" library="adafruit" deviceset="LED" device="CHIPLED_0805" value="Green">
 <attribute name="MF" value=""/>
@@
 <part name="C8" library="SparkFun-Passives" deviceset="CAP" device="0805" value="0.1uF"/>
 <part name="U3" library="ATMEGA328P-MU" deviceset="ATMEGA328P-MU" device=""/>
+<part name="U$1" library="ftdi_ft231xq-r" deviceset="FT231XQ-R" device=""/>
 </parts>
 <sheets>
@@
 <text x="142.24" y="-152.4" size="5.08" layer="94" font="vector" ratio="20">CRT Labs</text>
 <text x="147.32" y="-157.48" size="2.54" layer="94" font="vector" ratio="10">Sensor Node</text>
-<text x="160.02" y="-167.64" size="2.54" layer="94" font="vector" ratio="10" align="bottom-center">v0.6
+<text x="160.02" y="-167.64" size="2.54" layer="94" font="vector" ratio="10" align="bottom-center">v0.8
 (October 2016)</text>
 <text x="160.02" y="-175.26" size="1.27" layer="94" font="vector" ratio="10" align="bottom-center">Designed by
@@
 <instance part="GND3" gate="1" x="149.86" y="-81.28"/>
 <instance part="J3" gate="G$1" x="238.76" y="-116.84" rot="R180"/>
-<instance part="U5" gate="U$1" x="299.72" y="-134.62"/>
 <instance part="RX" gate="G$1" x="332.74" y="-144.78" rot="R270">
 <attribute name="OC_NEWARK" x="332.74" y="-144.78" size="1.778" layer="96" rot="R90" display="off"/>
@@
 <instance part="C8" gate="G$1" x="124.46" y="33.02" rot="R180"/>
 <instance part="U3" gate="G$1" x="304.8" y="91.44"/>
+<instance part="U$1" gate="G$1" x="302.26" y="-134.62"/>
 </instances>
 <busses>
@@
 </segment>
 <segment>
-<pinref part="U5" gate="U$1" pin="GND@6"/>
 <wire x1="287.02" y1="-147.32" x2="284.48" y2="-147.32" width="0.1524" layer="91"/>
 <wire x1="284.48" y1="-147.32" x2="284.48" y2="-149.86" width="0.1524" layer="91"/>
-<pinref part="U5" gate="U$1" pin="GND@16"/>
 <wire x1="287.02" y1="-149.86" x2="284.48" y2="-149.86" width="0.1524" layer="91"/>
 <wire x1="284.48" y1="-149.86" x2="284.48" y2="-157.48" width="0.1524" layer="91"/>
 <junction x="284.48" y="-149.86"/>
 <pinref part="GND10" gate="1" pin="GND"/>
+<pinref part="U$1" gate="G$1" pin="GND_3"/>
+<pinref part="U$1" gate="G$1" pin="GND_13"/>
+<pinref part="U$1" gate="G$1" pin="GND_21"/>
+<wire x1="287.02" y1="-144.78" x2="284.48" y2="-144.78" width="0.1524" layer="91"/>
+<wire x1="284.48" y1="-144.78" x2="284.48" y2="-147.32" width="0.1524" layer="91"/>
+<junction x="284.48" y="-147.32"/>
 </segment>
 <segment>
@@
 </segment>
 <segment>
-<pinref part="U5" gate="U$1" pin="!DTR"/>
-<wire x1="312.42" y1="-132.08" x2="322.58" y2="-132.08" width="0.1524" layer="91"/>
 <label x="322.58" y="-132.08" size="1.778" layer="95" xref="yes"/>
+<pinref part="U$1" gate="G$1" pin="DTR#"/>
+<wire x1="317.5" y1="-132.08" x2="322.58" y2="-132.08" width="0.1524" layer="91"/>
 </segment>
 </net>
@@
 </segment>
 <segment>
-<pinref part="U5" gate="U$1" pin="TXD"/>
-<wire x1="312.42" y1="-119.38" x2="322.58" y2="-119.38" width="0.1524" layer="91"/>
 <label x="322.58" y="-119.38" size="1.778" layer="95" xref="yes"/>
+<pinref part="U$1" gate="G$1" pin="TXD"/>
+<wire x1="317.5" y1="-119.38" x2="322.58" y2="-119.38" width="0.1524" layer="91"/>
 </segment>
 </net>
@@
 </segment>
 <segment>
-<pinref part="U5" gate="U$1" pin="RXD"/>
-<wire x1="312.42" y1="-121.92" x2="322.58" y2="-121.92" width="0.1524" layer="91"/>
 <label x="322.58" y="-121.92" size="1.778" layer="95" xref="yes"/>
+<pinref part="U$1" gate="G$1" pin="RXD"/>
+<wire x1="317.5" y1="-121.92" x2="322.58" y2="-121.92" width="0.1524" layer="91"/>
 </segment>
 </net>
@@
 <net name="N$25" class="0">
 <segment>
-<pinref part="U5" gate="U$1" pin="USBDM"/>
 <wire x1="287.02" y1="-129.54" x2="271.78" y2="-129.54" width="0.1524" layer="91"/>
 <wire x1="271.78" y1="-129.54" x2="271.78" y2="-139.7" width="0.1524" layer="91"/>
 <wire x1="271.78" y1="-139.7" x2="266.7" y2="-139.7" width="0.1524" layer="91"/>
 <pinref part="R21" gate="G$1" pin="1"/>
+<pinref part="U$1" gate="G$1" pin="USBDM"/>
 </segment>
 </net>
 <net name="N$26" class="0">
 <segment>
-<pinref part="U5" gate="U$1" pin="USBDP"/>
 <wire x1="287.02" y1="-132.08" x2="274.32" y2="-132.08" width="0.1524" layer="91"/>
 <wire x1="274.32" y1="-132.08" x2="274.32" y2="-142.24" width="0.1524" layer="91"/>
 <wire x1="274.32" y1="-142.24" x2="266.7" y2="-142.24" width="0.1524" layer="91"/>
 <pinref part="R12" gate="G$1" pin="1"/>
+<pinref part="U$1" gate="G$1" pin="USBDP"/>
 </segment>
 </net>
 <net name="N$17" class="0">
 <segment>
-<pinref part="U5" gate="U$1" pin="CBUS1"/>
 <pinref part="RX" gate="G$1" pin="C"/>
-<wire x1="312.42" y1="-144.78" x2="327.66" y2="-144.78" width="0.1524" layer="91"/>
+<pinref part="U$1" gate="G$1" pin="CBUS1"/>
+<wire x1="317.5" y1="-144.78" x2="327.66" y2="-144.78" width="0.1524" layer="91"/>
 </segment>
 </net>
 <net name="N$18" class="0">
 <segment>
-<pinref part="U5" gate="U$1" pin="CBUS2"/>
 <pinref part="TX" gate="G$1" pin="C"/>
-<wire x1="312.42" y1="-147.32" x2="320.04" y2="-147.32" width="0.1524" layer="91"/>
+<pinref part="U$1" gate="G$1" pin="CBUS2"/>
+<wire x1="317.5" y1="-147.32" x2="320.04" y2="-147.32" width="0.1524" layer="91"/>
 </segment>
 </net>
@@
 <net name="VBUS" class="0">
 <segment>
-<pinref part="U5" gate="U$1" pin="VCC"/>
 <pinref part="C11" gate="G$1" pin="1"/>
 <wire x1="287.02" y1="-119.38" x2="261.62" y2="-119.38" width="0.1524" layer="91"/>
@@
 <pinref part="J3" gate="G$1" pin="VBUS"/>
 <wire x1="241.3" y1="-119.38" x2="261.62" y2="-119.38" width="0.1524" layer="91"/>
+<pinref part="U$1" gate="G$1" pin="VCC"/>
 </segment>
 </net>
@@
 <net name="FTDI_VCC" class="0">
 <segment>
-<pinref part="U5" gate="U$1" pin="!RESET"/>
 <wire x1="287.02" y1="-137.16" x2="281.94" y2="-137.16" width="0.1524" layer="91"/>
 <wire x1="281.94" y1="-137.16" x2="281.94" y2="-124.46" width="0.1524" layer="91"/>
-<pinref part="U5" gate="U$1" pin="3V3OUT"/>
 <wire x1="281.94" y1="-124.46" x2="287.02" y2="-124.46" width="0.1524" layer="91"/>
-<pinref part="U5" gate="U$1" pin="VCCIO"/>
 <wire x1="287.02" y1="-124.46" x2="287.02" y2="-121.92" width="0.1524" layer="91"/>
+<wire x1="287.02" y1="-121.92" x2="279.4" y2="-121.92" width="0.1524" layer="91"/>
+<label x="279.4" y="-121.92" size="1.778" layer="95" rot="R180" xref="yes"/>
+<pinref part="U$1" gate="G$1" pin="3V3OUT"/>
 <junction x="287.02" y="-124.46"/>
-<wire x1="287.02" y1="-121.92" x2="279.4" y2="-121.92" width="0.1524" layer="91"/>
+<pinref part="U$1" gate="G$1" pin="RESET#"/>
+<pinref part="U$1" gate="G$1" pin="VCCIO"/>
 <junction x="287.02" y="-121.92"/>
-<label x="279.4" y="-121.92" size="1.778" layer="95" rot="R180" xref="yes"/>
-</segment>
-<segment>
+</segment>
+<segment>
