File: hardware/v0.54/sensor_board_v0.54.sch (EAGLE design)
At the start: 59 parts, among them J3 USB-MICROB, J6 AVR_SPI_PRG_6PTH, U1 ATMEGA328P, U10 TSL2591, U3 OPA344, U4 RFM69HW, U5 FT231XS, U6 ADMP401, U8 MCP1703CB, U9 BMP280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

Commit message: BOM update
- Added MPN for 0.1 and 10uF
- Added I2C address and value for SHT35 on schematic
Parts:
- C4: MPN CC0805ZRY5V8BB105 -> CC0805KKX5R6BB106
- C6: MPN CC0805ZRY5V8BB105 -> CC0805KRX7R9BB104
- U2: value (none) -> SHT35
Connections:
- removed net A7: U1.ADC7
- removed net D5: U1.PD5(T1)
Other:
- note added: "0x44"
Changed lines of the file:
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@@
 </part>
 <part name="C6" library="SparkFun-Capacitors" deviceset="CAP" device="0805" value="0.1uF">
-<attribute name="MPN" value="CC0805ZRY5V8BB105"/>
+<attribute name="MPN" value="CC0805KRX7R9BB104"/>
 </part>
 <part name="GND2" library="SparkFun-Aesthetics" deviceset="GND" device=""/>
@@
 <part name="J4" library="SparkFun-Connectors" deviceset="M02" device="PTH"/>
 <part name="J5" library="SparkFun-Connectors" deviceset="M02" device="PTH"/>
-<part name="U2" library="Adafruit SHT31" deviceset="SHT3X" device="">
+<part name="U2" library="Adafruit SHT31" deviceset="SHT3X" device="" value="SHT35">
 <attribute name="MPN" value="SHT35-DIS-B"/>
 </part>
@@
 </part>
 <part name="C4" library="SparkFun-Capacitors" deviceset="CAP" device="0805" value="10uF">
-<attribute name="MPN" value="CC0805ZRY5V8BB105"/>
+<attribute name="MPN" value="CC0805KKX5R6BB106"/>
 </part>
 <part name="C3" library="SparkFun-Capacitors" deviceset="CAP" device="0805" value="1uF">
@@
 Serial</text>
 <text x="170.18" y="-15.24" size="3.81" layer="94">PM2.5 sensor</text>
+<text x="251.46" y="-7.62" size="1.778" layer="97">0x44</text>
 </plain>
 <instances>
@@
 </segment>
 </net>
-<net name="D5" class="0">
-<segment>
-<pinref part="U1" gate="U$1" pin="PD5(T1)"/>
-<wire x1="261.62" y1="76.2" x2="269.24" y2="76.2" width="0.1524" layer="91"/>
-<label x="269.24" y="76.2" size="1.778" layer="95" xref="yes"/>
-</segment>
-</net>
 <net name="N$4" class="0">
 <segment>
@@
 </segment>
 </net>
-<net name="A7" class="0">
-<segment>
-<pinref part="U1" gate="U$1" pin="ADC7"/>
-<wire x1="261.62" y1="93.98" x2="269.24" y2="93.98" width="0.1524" layer="91"/>
-<label x="269.24" y="93.98" size="1.778" layer="95" xref="yes"/>
-</segment>
-</net>
 <net name="A0" class="0">
 <segment>
@@
 </sheet>
 </sheets>
+<errors>
+</errors>
 </schematic>
 </drawing>

Commit message: v0.54 update - resonator library changed
- Replaced previous resonator library (thinner pads, incorrectly
aligned, usually got lucky) with one that has fatter pads (from RFM69
USB gateway)
Parts:
- removed Y1: 16MHZ, SparkFun-FreqCtrl:RESONATOR16MHZ
- added X1: 16 MHz, SparkFun:RESONATORSMD
Connections:
- net GND: now also X1.2; no longer Y1.2
- net N$4: now also X1.3; no longer Y1.3
- net N$5: now also X1.1; no longer Y1.1
Changed lines of the file:
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@@
 <?xml version="1.0" encoding="utf-8"?>
 <!DOCTYPE eagle SYSTEM "eagle.dtd">
-<eagle version="7.7.0">
+<eagle version="8.1.0">
 <drawing>
 <settings>
@@
 <class number="0" name="default" width="0" drill="0">
 </class>
+<class number="1" name="power" width="0.381" drill="0">
+<clearance class="1" value="0.254"/>
+</class>
 </classes>
 <parts>
@@
 <part name="C5" library="SparkFun-Passives" deviceset="CAP" device="0805" value="0.1uF">
 <attribute name="MPN" value="CC0805KRX7R9BB104"/>
-</part>
-<part name="Y1" library="SparkFun-FreqCtrl" deviceset="RESONATOR" device="16MHZ" value="16MHZ">
-<attribute name="MF" value=""/>
-<attribute name="MPN" value="CSTCE16M0V53-R0"/>
-<attribute name="OC_NEWARK" value="unknown"/>
 </part>
 <part name="SUPPLY7" library="SparkFun-Aesthetics" deviceset="VCC" device=""/>
@@
 <attribute name="MPN" value="CC0805ZRY5V8BB105"/>
 </part>
+<part name="X1" library="SparkFun" deviceset="RESONATOR" device="SMD" value="16 MHz"/>
 </parts>
 <sheets>
@@
 <attribute name="MPN" x="269.24" y="-60.96" size="1.778" layer="96" rot="R270" display="off"/>
 </instance>
-<instance part="Y1" gate="G$1" x="208.28" y="76.2">
-<attribute name="OC_NEWARK" x="208.28" y="76.2" size="1.778" layer="96" rot="R270" display="off"/>
-<attribute name="MF" x="208.28" y="76.2" size="1.778" layer="96" rot="R270" display="off"/>
-<attribute name="MPN" x="208.28" y="76.2" size="1.778" layer="96" rot="R270" display="off"/>
-</instance>
 <instance part="SUPPLY7" gate="G$1" x="279.4" y="121.92"/>
 <instance part="U8" gate="G$1" x="-17.78" y="50.8">
@@
 <attribute name="MPN" x="111.76" y="-2.54" size="1.778" layer="96" rot="R270" display="off"/>
 </instance>
+<instance part="X1" gate="G$1" x="208.28" y="76.2"/>
 </instances>
 <busses>
@@
 <wire x1="208.28" y1="60.96" x2="208.28" y2="58.42" width="0.1524" layer="91"/>
 <junction x="208.28" y="58.42"/>
-<pinref part="Y1" gate="G$1" pin="2"/>
 <wire x1="208.28" y1="68.58" x2="208.28" y2="60.96" width="0.1524" layer="91"/>
 <junction x="208.28" y="60.96"/>
@@
 <wire x1="193.04" y1="73.66" x2="193.04" y2="60.96" width="0.1524" layer="91"/>
 <wire x1="193.04" y1="60.96" x2="208.28" y2="60.96" width="0.1524" layer="91"/>
+<pinref part="X1" gate="G$1" pin="2"/>
 </segment>
 <segment>
@@
 <segment>
 <pinref part="U1" gate="U$1" pin="PB7(XTAL2/TOSC2)"/>
-<pinref part="Y1" gate="G$1" pin="3"/>
 <wire x1="213.36" y1="81.28" x2="210.82" y2="81.28" width="0.1524" layer="91"/>
 <wire x1="210.82" y1="81.28" x2="210.82" y2="76.2" width="0.1524" layer="91"/>
+<pinref part="X1" gate="G$1" pin="3"/>
 </segment>
 </net>
@@
 <segment>
 <pinref part="U1" gate="U$1" pin="PB6(XTAL1/TOSC1)"/>
-<pinref part="Y1" gate="G$1" pin="1"/>
 <wire x1="213.36" y1="86.36" x2="205.74" y2="86.36" width="0.1524" layer="91"/>
 <wire x1="205.74" y1="86.36" x2="205.74" y2="76.2" width="0.1524" layer="91"/>
+<pinref part="X1" gate="G$1" pin="1"/>
 </segment>
 </net>
