File: hardware/v0.55/sensor_board_v0.55.brd (EAGLE design)
At the start: 56.4 x 41.9 mm, 60 parts, among them J3 USB-MICROB, J6 AVR_SPI_PRG_6PTH, U1 ATMEGA328P, U10 TSL2591, U11 915MHz, U2 SHT35, U3 OPA344, U5 FT231XS, U6 ADMP401, U7 PMS7003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

Commit message: Silkscreen updates
Other:
- board text added: "Designed by Akram Ali"
- board text added: "v0.55b | May 2017"
- board text removed: "Designed by Akram Ali and Dave Conroy"
- board text removed: "v0.55 | April 2017"
Changed lines of the file:
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@@
 <plain>
 <text x="36.6268" y="10.9728" size="1.016" layer="122" font="vector" ratio="16" rot="MR0" align="center-left">Touchstone</text>
-<text x="50.546" y="6.7056" size="0.6096" layer="122" font="vector" rot="MR0">Designed by Akram Ali and Dave Conroy</text>
-<text x="36.5506" y="9.525" size="0.6096" layer="122" font="vector" rot="MR0">v0.55 | April 2017</text>
+<text x="50.546" y="6.7056" size="0.6096" layer="122" font="vector" rot="MR0">Designed by Akram Ali</text>
+<text x="36.5506" y="9.525" size="0.6096" layer="122" font="vector" rot="MR0">v0.55b | May 2017</text>
 <text x="36.5506" y="9.144" size="0.8128" layer="122" font="vector" ratio="12" rot="MR180" align="bottom-right">crtlabs.org</text>
 <rectangle x1="43.4086" y1="8.3566" x2="43.815" y2="8.4074" layer="122" rot="R180"/>
