File: hardware/v0.55/sensor_board_v0.55.sch (EAGLE design)
At the start: 60 parts, among them J3 USB-MICROB, J6 AVR_SPI_PRG_6PTH, U1 ATMEGA328P, U10 TSL2591, U11 915MHz, U2 SHT35, U3 OPA344, U5 FT231XS, U6 ADMP401, U7 PMS7003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

Commit message: Silkscreen updates
Other:
- note added: "0.55b"
- note removed: "0.55"
Changed lines of the file:
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@@
 <text x="246.38" y="-78.74" size="1.778" layer="97">0x5A</text>
 <text x="160.02" y="20.32" size="1.778" layer="97">0x77</text>
-<text x="257.556" y="-102.362" size="2.54" layer="94" font="vector" ratio="10">0.55</text>
+<text x="257.556" y="-102.362" size="2.54" layer="94" font="vector" ratio="10">0.55b</text>
 <text x="192.786" y="-107.442" size="2.54" layer="94" font="vector" ratio="10">github.crtlabs.org</text>
 <text x="73.66" y="30.48" size="1.778" layer="97">0x29</text>
